Commit message: fix(sensor_kit): match MORAI sensor frame_ids (lidar/imu)
MORAI 가 /lidar/points 에 header.frame_id="lidar", /Imu 에 "imu" 를 박는 것을
실측 확인. description 의 프레임명이 velodyne_top/imu_link 라 TF(base_link->센서)가
안 맞아 lidar crop box 변환이 실패했음. 프레임명을 MORAI 가 박는 lidar/imu 로
맞춰 base_link->lidar, base_link->imu TF 가 성립하게 함. gnss 는 변환 노드가
frame_id 를 gnss_link 로 강제하므로 그대로 둠.

File: src/launcher/autoware_launch/sensor_kit/morai_sensor_kit_launch/morai_sensor_kit_description/urdf/sensor_kit.xacro (robot description, xacro)
@@ -1,4 +1,4 @@
 <?xml version="1.0"?>
-<!-- MORAI sensor kit 의 센서 프레임(velodyne_top/imu_link/gnss_link)을 정의하는 최소 xacro 매크로 -->
+<!-- MORAI sensor kit 의 센서 프레임(lidar/imu/gnss_link)을 정의하는 최소 xacro 매크로 -->
 <robot xmlns:xacro="http://ros.org/wiki/xacro">
   <xacro:macro name="sensor_kit_macro" params="parent x y z roll pitch yaw">
@@ -13,29 +13,29 @@
     <link name="${sensor_kit_base_link}"/>
     <!-- LiDAR -->
-    <joint name="velodyne_top_joint" type="fixed">
+    <joint name="lidar_joint" type="fixed">
       <origin
-        xyz="${calibration['sensor_kit_base_link']['velodyne_top']['x']}
-             ${calibration['sensor_kit_base_link']['velodyne_top']['y']}
-             ${calibration['sensor_kit_base_link']['velodyne_top']['z']}"
-        rpy="${calibration['sensor_kit_base_link']['velodyne_top']['roll']}
-             ${calibration['sensor_kit_base_link']['velodyne_top']['pitch']}
-             ${calibration['sensor_kit_base_link']['velodyne_top']['yaw']}"/>
+        xyz="${calibration['sensor_kit_base_link']['lidar']['x']}
+             ${calibration['sensor_kit_base_link']['lidar']['y']}
+             ${calibration['sensor_kit_base_link']['lidar']['z']}"
+        rpy="${calibration['sensor_kit_base_link']['lidar']['roll']}
+             ${calibration['sensor_kit_base_link']['lidar']['pitch']}
+             ${calibration['sensor_kit_base_link']['lidar']['yaw']}"/>
       <parent link="${sensor_kit_base_link}"/>
-      <child link="velodyne_top"/>
+      <child link="lidar"/>
     </joint>
-    <link name="velodyne_top"/>
+    <link name="lidar"/>
     <!-- IMU -->
-    <joint name="imu_link_joint" type="fixed">
+    <joint name="imu_joint" type="fixed">
       <origin
-        xyz="${calibration['sensor_kit_base_link']['imu_link']['x']}
-             ${calibration['sensor_kit_base_link']['imu_link']['y']}
-             ${calibration['sensor_kit_base_link']['imu_link']['z']}"
-        rpy="${calibration['sensor_kit_base_link']['imu_link']['roll']}
-             ${calibration['sensor_kit_base_link']['imu_link']['pitch']}
-             ${calibration['sensor_kit_base_link']['imu_link']['yaw']}"/>
+        xyz="${calibration['sensor_kit_base_link']['imu']['x']}
+             ${calibration['sensor_kit_base_link']['imu']['y']}
+             ${calibration['sensor_kit_base_link']['imu']['z']}"
+        rpy="${calibration['sensor_kit_base_link']['imu']['roll']}
+             ${calibration['sensor_kit_base_link']['imu']['pitch']}
+             ${calibration['sensor_kit_base_link']['imu']['yaw']}"/>
       <parent link="${sensor_kit_base_link}"/>
-      <child link="imu_link"/>
+      <child link="imu"/>
     </joint>
-    <link name="imu_link"/>
+    <link name="imu"/>
     <!-- GNSS -->
     <joint name="gnss_link_joint" type="fixed">
